File: EDA/cm4-carrier/cm4-carrier.kicad_pcb (KiCad board)
At the start: 2 copper layers, 68.6 x 150 mm, 12 parts, among them J1 35RAPC4BHN2, J4 Conn_01x22_Female, J5 Conn_01x22_Female, J6 USB4105-GF-A, U1 Flash-LED-Lumiled

Commit message: update EDA files
Parts:
- added J2: FH72-31S-0.3SHW, SPIRIT-footprints:HRS_FH72-31S-0.3SHW, F.Cu at (72.4, 166.4)
- added J3: 10pinFPC, SPIRIT-footprints:10PIN, F.Cu at (30.5, 95.2)
- added MK1: microphone, SPIRIT-footprints:microphone_SPH0645LM4H-B, F.Cu at (73.7, 174.8)
- added REF**: 720pLCD, SPIRIT-footprints:720pLCD, F.Cu at (49.9, 36.6)
- added REF**: fingerprintSEN-17151, SPIRIT-footprints:fingerSEN-17151, F.Cu at (22.7, 135.9)
- added SW1: VOL-, SPIRIT-footprints:buttonSW_TL3330_EWI, F.Cu at (52.1, 49.5)
- added SW2: PROG, SPIRIT-footprints:buttonSW_TL3330_EWI, F.Cu at (52.1, 77.5)
- added SW3: VOL+, SPIRIT-footprints:buttonSW_TL3330_EWI, F.Cu at (52.1, 59.7)
- added SW4: POW, SPIRIT-footprints:buttonSW_TL3330_EWI, F.Cu at (127.0, 54.6)
- J5: moved to F.Cu
- moved J5 78.4 mm to (29.1, 116.8)
- moved J4 53.7 mm to (94.0, 36.8), turned to 180 degrees
- moved R1 52.1 mm to (29.2, 104.1)
- moved J1 28.0 mm to (58.4, 169.7)
- moved Module1 24.2 mm to (68.7, 44.0)
- moved REF** 24.2 mm to (102.1, 60.0)
- moved CR1 22.1 mm to (97.8, 172.7)
- moved J6 22.1 mm to (89.8, 174.8)
- moved U1 15.4 mm to (74.0, 32.2)
- moved BAT1 15.4 mm to (81.3, 167.1)
- moved LS3 15.4 mm to (114.3, 32.5)
- moved LS4 14.1 mm to (118.1, 172.2)
Other:
- board size 68.6 x 150 mm -> 80 x 150 mm

Commit message: update files
Parts:
- removed the J4 at (94.0, 36.8)
- removed the J5 at (29.1, 116.8)
- added B1: VIBR, SPIRIT-footprints:VIBRATION-PUI_HD-EMB1205-3-SC-R, F.Cu at (63.5, 127.0)
- added G***: LOGO, LOGO, F.Cu at (77.5, 108.0)
- added G***: LOGO, LOGO, F.Cu at (67.3, 111.8)
- added J1: Conn_01x22_Female, SPIRIT-footprints:Hirose_FH12-22S-0.5SH_1x22-1MP_P0.50mm_Horizontal, F.Cu at (69.8, 61.6)
- added U2: CHARGER-BQ24161YFFR, SPIRIT-footprints:CHARGER-YFF49, F.Cu at (36.8, 111.8)
- added U3: BAT-MONITOR-BQ27530YZFT-G1, SPIRIT-footprints:BAT-MONITOR-YZF15_TEX, F.Cu at (43.8, 117.3)
- added U4: STABILIZER-MC34063ADR, SPIRIT-footprints:STABILIZER-MC34063ADR, F.Cu at (26.7, 113.0)
- added U5: BAT-CONNECTOR-FLTS22WR00, SPIRIT-footprints:BAT-CONNECTOR-FLTS22WR00, F.Cu at (76.0, 147.6)
- added U6: GPS-moduleYIC31009EBGG, SPIRIT-footprints:GPS-moduleYIC31009EBGG, F.Cu at (61.6, 144.1)
- J5: renamed from J3; value 10pinFPC -> FINGER
- REF**: moved to B.Cu
- moved REF** 96.9 mm to (104.3, 83.7), turned to 180 degrees
- moved J5 40.9 mm to (71.1, 90.8), turned to -90 degrees
- moved REF** 28.9 mm to (24.0, 49.3)
- moved U1 22.0 mm to (95.9, 33.7)
- moved SW4 8.54 mm to (133.3, 60.3)
- moved LS1 7.08 mm to (121.3, 33.7)
- moved J4 7.00 mm to (65.4, 170.2)
- moved Module1 6.38 mm to (75.1, 44.6)
- moved MK1 6.38 mm to (80.0, 175.4)
- moved SW2 6.38 mm to (58.4, 78.1)
- moved SW3 6.38 mm to (58.4, 60.3)
- moved SW1 6.38 mm to (58.4, 50.2)
- moved REF** 6.38 mm to (108.4, 60.6)
- moved BAT1 6.38 mm to (87.6, 167.8)
- moved CR1 6.38 mm to (104.1, 173.4)
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- renumbered J6 to J2, J2 to J3, J1 to J4, LS3 to LS1, LS4 to LS2
Other:
- board size 80 x 150 mm -> 80 x 148.2 mm
- board text added: "V ELECTRONICS"

Commit message: update EDA
Parts:
- added D1: LED-INDICATOR, SPIRIT-footprints:LED-INDICATOR, F.Cu at (74.4, 161.9)
- added J6: SIM-G85D1160022HHR, SPIRIT-footprints:SIM-AMPHENOL_G85D1160022HHR, F.Cu at (196.8, 125.7)
- added S1: DIPSWITCH, SPIRIT-footprints:DIPSWITC-SW_219-4MST, F.Cu at (63.5, 143.5)
- added U8: DAC-TLV320DAC3100IRHBR, SPIRIT-footprints:DAC-IC_ADS125H01IRHBT, F.Cu at (83.8, 127.6)
- J4: value 35RAPC4BHN2 -> 35mmJACK-TRRS; footprint SPIRIT-footprints:35mm-jack-35RAPC4BHN2-switchcraft -> SPIRIT-footprints:35mmJACK-TRRS
- U2: value CHARGER-BQ24161YFFR -> CHARGER-SWITCHER-BQ25303JRTER; footprint SPIRIT-footprints:CHARGER-YFF49 -> SPIRIT-footprints:CHARGER-SWITCHER-RTE0016C
- U4: value STABILIZER-MC34063ADR -> BAT-STEP-UP-MIC2876-5.0YMT-TR; footprint SPIRIT-footprints:STABILIZER-MC34063ADR -> SPIRIT-footprints:BAT-STEP-UP-UDFN8_2X2_MCH
- U6: value GPS-moduleYIC31009EBGG -> GSM-GPS-EC25VFA-512-STD; footprint SPIRIT-footprints:GPS-moduleYIC31009EBGG -> SPIRIT-footprints:GSM-GPS-XCVR_EC25VFA-512-STD
- moved BAT1 160.3 mm to (235.6, 106.0), turned to 180 degrees
- moved U6 107.0 mm to (168.3, 136.5)
- moved U4 77.0 mm to (87.6, 160.0)
- moved U2 61.3 mm to (91.4, 139.7)
- moved U3 57.7 mm to (91.4, 149.9)
- moved REF** 34.5 mm to (55.9, 36.2)
- moved G*** 1.91 mm to (79.4, 108.0)
- moved G*** 1.91 mm to (69.2, 111.8)
- moved J4 0.64 mm to (66.0, 170.2), turned to 90 degrees

Commit message: update EDA
Parts:
- removed J4: 35mmJACK-TRRS, SPIRIT-footprints:35mmJACK-TRRS
- added J3: CAM FPC15pins05pitch, SPIRIT-footprints:FPC15pins05pitch, F.Cu at (67.3, 61.0)
- added R2: 5.1kOhm, SPIRIT-footprints:CC-PULLDOWN-RESISOTR, F.Cu at (89.5, 175.9)
- added R3: 5.1kOhm, SPIRIT-footprints:CC-PULLDOWN-RESISOTR, F.Cu at (89.5, 172.2)
- J1: value Conn_01x22_Female -> SJ2-35894B-SMT-TR; footprint SPIRIT-footprints:Hirose_FH12-22S-0.5SH_1x22-1MP_P0.50mm_Horizontal -> SPIRIT-footprints:35mmJACK-CUI_SJ2-35894B-SMT-TR
- U6: moved to B.Cu
- moved BAT1 161.7 mm to (86.8, 169.4), turned to 90 degrees
- moved J6 132.6 mm to (64.8, 114.3), turned to -90 degrees
- moved J1 108.4 mm to (67.0, 169.9), turned to 90 degrees
- moved G*** 79.5 mm to (106.0, 33.0)
- moved U6 75.0 mm to (95.2, 119.4), turned to 180 degrees
- moved G*** 43.2 mm to (26.0, 111.8)
- renumbered J3 to DIS1
Connections:
- B1 pad N: unconnected-(B1-PadN) -> GND
- B1 pad P: unconnected-(B1-PadP) -> Net-(B1-PadP)
- CR1 pad 1: unconnected-(CR1-Pad1) -> Net-(CR1-Pad1)
- CR1 pad 2: unconnected-(CR1-Pad2) -> Net-(CR1-Pad2)
- J1 pad 10: unconnected-(J1-Pad10) -> JACK-IN
- J2 pad A4_B9: unconnected-(J2-PadA4_B9) -> Net-(CR1-Pad1)
- J2 pad A5: unconnected-(J2-PadA5) -> Net-(J2-PadA5)
- J2 pad B1_A12: unconnected-(J2-PadB1_A12) -> GND
- J2 pad B4_A9: unconnected-(J2-PadB4_A9) -> Net-(CR1-Pad1)
- J2 pad B5: unconnected-(J2-PadB5) -> Net-(J2-PadB5)
- J2 pad B6: unconnected-(J2-PadB6) -> D+
- J2 pad B7: unconnected-(J2-PadB7) -> D-
- J2 pad SH1: unconnected-(J2-PadSH1) -> GND
- J2 pad SH2: unconnected-(J2-PadSH2) -> GND
- J2 pad SH3: unconnected-(J2-PadSH3) -> GND
- J2 pad SH4: unconnected-(J2-PadSH4) -> GND
- J6 pad C5: unconnected-(J6-PadC5) -> GND
- J6 pad S1: unconnected-(J6-PadS1) -> GND
- J6 pad S2: unconnected-(J6-PadS2) -> GND
- J6 pad S3: unconnected-(J6-PadS3) -> GND
- MK1 pad 5: unconnected-(MK1-Pad5) -> MIC-SWITCH
- Module1 pad 1: unconnected-(Module1-Pad1) -> GND
- Module1 pad 108: unconnected-(Module1-Pad108) -> GND
- Module1 pad 113: unconnected-(Module1-Pad113) -> GND
- Module1 pad 114: unconnected-(Module1-Pad114) -> GND
- Module1 pad 119: unconnected-(Module1-Pad119) -> GND
- Module1 pad 120: unconnected-(Module1-Pad120) -> GND
- Module1 pad 125: unconnected-(Module1-Pad125) -> GND
- Module1 pad 126: unconnected-(Module1-Pad126) -> GND
- Module1 pad 13: unconnected-(Module1-Pad13) -> GND
- Module1 pad 131: unconnected-(Module1-Pad131) -> GND
- Module1 pad 132: unconnected-(Module1-Pad132) -> GND
- Module1 pad 137: unconnected-(Module1-Pad137) -> GND
- Module1 pad 138: unconnected-(Module1-Pad138) -> GND
- Module1 pad 14: unconnected-(Module1-Pad14) -> GND
- Module1 pad 144: unconnected-(Module1-Pad144) -> GND
- Module1 pad 150: unconnected-(Module1-Pad150) -> GND
- Module1 pad 155: unconnected-(Module1-Pad155) -> GND
- Module1 pad 156: unconnected-(Module1-Pad156) -> GND
- Module1 pad 161: unconnected-(Module1-Pad161) -> GND
- Module1 pad 162: unconnected-(Module1-Pad162) -> GND
- Module1 pad 167: unconnected-(Module1-Pad167) -> GND
- Module1 pad 168: unconnected-(Module1-Pad168) -> GND
- Module1 pad 173: unconnected-(Module1-Pad173) -> GND
- Module1 pad 174: unconnected-(Module1-Pad174) -> GND
- Module1 pad 179: unconnected-(Module1-Pad179) -> GND
- Module1 pad 180: unconnected-(Module1-Pad180) -> GND
- Module1 pad 185: unconnected-(Module1-Pad185) -> GND
- Module1 pad 186: unconnected-(Module1-Pad186) -> GND
- Module1 pad 191: unconnected-(Module1-Pad191) -> GND
- Module1 pad 192: unconnected-(Module1-Pad192) -> GND
- Module1 pad 197: unconnected-(Module1-Pad197) -> GND
- Module1 pad 198: unconnected-(Module1-Pad198) -> GND
- Module1 pad 2: unconnected-(Module1-Pad2) -> GND
- Module1 pad 22: unconnected-(Module1-Pad22) -> GND
- Module1 pad 23: unconnected-(Module1-Pad23) -> GND
- Module1 pad 32: unconnected-(Module1-Pad32) -> GND
- Module1 pad 33: unconnected-(Module1-Pad33) -> GND
- Module1 pad 42: unconnected-(Module1-Pad42) -> GND
- Module1 pad 43: unconnected-(Module1-Pad43) -> GND
- Module1 pad 46: unconnected-(Module1-Pad46) -> Net-(Module1-Pad46)
- Module1 pad 48: unconnected-(Module1-Pad48) -> Net-(B1-PadP)
- Module1 pad 50: unconnected-(Module1-Pad50) -> Net-(Module1-Pad50)
- Module1 pad 52: unconnected-(Module1-Pad52) -> GND
- Module1 pad 53: unconnected-(Module1-Pad53) -> GND
- Module1 pad 54: unconnected-(Module1-Pad54) -> Net-(Module1-Pad54)
- Module1 pad 56: unconnected-(Module1-Pad56) -> Net-(Module1-Pad56)
- Module1 pad 58: unconnected-(Module1-Pad58) -> Net-(Module1-Pad58)
- Module1 pad 60: unconnected-(Module1-Pad60) -> GND
- Module1 pad 66: unconnected-(Module1-Pad66) -> GND
- Module1 pad 71: unconnected-(Module1-Pad71) -> GND
- Module1 pad 74: unconnected-(Module1-Pad74) -> GND
- Module1 pad 8: unconnected-(Module1-Pad8) -> GND
- Module1 pad 98: unconnected-(Module1-Pad98) -> GND
- S1 pad 1: unconnected-(S1-Pad1) -> Net-(S1-Pad1)
- S1 pad 2: unconnected-(S1-Pad2) -> Net-(S1-Pad1)
- S1 pad 3: unconnected-(S1-Pad3) -> Net-(S1-Pad1)
- S1 pad 4: unconnected-(S1-Pad4) -> Net-(S1-Pad1)
- S1 pad 5: unconnected-(S1-Pad5) -> PWR-KILL
- S1 pad 6: unconnected-(S1-Pad6) -> GPSGSM-SWITCH
- S1 pad 7: unconnected-(S1-Pad7) -> CAM-SWITCH
- S1 pad 8: unconnected-(S1-Pad8) -> MIC-SWITCH
- SW1 pad 1: unconnected-(SW1-Pad1) -> VCC
- SW1 pad 2: unconnected-(SW1-Pad2) -> Net-(Module1-Pad54)
- SW2 pad 1: unconnected-(SW2-Pad1) -> VCC
- SW2 pad 2: unconnected-(SW2-Pad2) -> Net-(Module1-Pad50)
- SW3 pad 1: unconnected-(SW3-Pad1) -> VCC
- SW3 pad 2: unconnected-(SW3-Pad2) -> Net-(Module1-Pad56)
- SW4 pad 1: unconnected-(SW4-Pad1) -> VCC
- SW4 pad 2: unconnected-(SW4-Pad2) -> Net-(Module1-Pad58)
- U1 pad 1: unconnected-(U1-Pad1) -> GND
- U1 pad 2: unconnected-(U1-Pad2) -> Net-(Module1-Pad46)
Other:
- board text added: "01"
- board text added: "Prototype unit"

Commit message: update EDA
Parts:
- removed CR1: SMBJ5.0A, SPIRIT-footprints:TVS-DO-214AASMB_J-BEND_LTF
- removed J3: CAM FPC15pins05pitch, SPIRIT-footprints:FPC15pins05pitch
- added TP1: test-pad-1, SPIRIT-footprints:test-pad-1, F.Cu at (66.0, 74.9)
- added TP2: test-pad-1, SPIRIT-footprints:test-pad-1, F.Cu at (69.2, 74.9)
- added TP3: test-pad-1, SPIRIT-footprints:test-pad-1, F.Cu at (109.9, 33.7)
- added TP4: test-pad-1, SPIRIT-footprints:test-pad-1, F.Cu at (71.8, 126.0)
- added TP5: test-pad-1, SPIRIT-footprints:test-pad-1, F.Cu at (78.1, 173.0)
- added TP6: test-pad-1, SPIRIT-footprints:test-pad-1, F.Cu at (83.2, 173.0)
- added U10: TVSdiode-array-TPD4EUSB30DQAR, SPIRIT-footprints:TVSdiode-arrayDQA10, F.Cu at (114.9, 162.4)
- added U7: FPC15pin-1mm-pitch-F52Q-1A7H1-11015, SPIRIT-footprints:FPC15pin-1mm-pitch-CONN_F52Q-1A7H1-11015_AMP, F.Cu at (66.9, 61.0)
- added U9: CODEC-TLV320AIC3204IRHBR, SPIRIT-footprints:CODEC-QFN50P500X500X100-33N, F.Cu at (112.4, 153.7)
- G***, S1: moved to B.Cu
- moved G*** 97.9 mm to (85.1, 33.7), turned to 180 degrees
- moved U8 54.3 mm to (122.6, 89.5)
- moved U2 25.1 mm to (95.2, 164.5)
- moved R1 15.8 mm to (39.4, 116.2)
- moved REF** 13.9 mm to (112.4, 74.0)
- moved D1 8.79 mm to (65.7, 161.3)
- moved MK1 6.40 mm to (73.6, 176.1)
- moved S1 5.12 mm to (64.1, 138.4), turned to -90 degrees
- moved Module1 4.51 mm to (79.5, 43.8)
- moved DIS1 1.42 mm to (79.4, 165.7)
- moved BAT1 0.23 mm to (87.0, 169.5)
- turned LS1 to 180 degrees
Connections:
- DIS1 pad 1: unconnected-(DIS1-Pad1) -> GND
- DIS1 pad 10: unconnected-(DIS1-Pad10) -> GND
- DIS1 pad 11: unconnected-(DIS1-Pad11) -> DSI1_C_N
- DIS1 pad 12: unconnected-(DIS1-Pad12) -> DSI1_C_P
- DIS1 pad 13: unconnected-(DIS1-Pad13) -> GND
- DIS1 pad 14: unconnected-(DIS1-Pad14) -> DSI1_D2_N
- DIS1 pad 15: unconnected-(DIS1-Pad15) -> DSI1_D2_P
- DIS1 pad 16: unconnected-(DIS1-Pad16) -> GND
- DIS1 pad 17: unconnected-(DIS1-Pad17) -> DSI1_D3_N
- DIS1 pad 18: unconnected-(DIS1-Pad18) -> DSI1_D3_P
- DIS1 pad 19: unconnected-(DIS1-Pad19) -> GND
- DIS1 pad 20: unconnected-(DIS1-Pad20) -> GND
- DIS1 pad 25: unconnected-(DIS1-Pad25) -> VCC
- DIS1 pad 26: unconnected-(DIS1-Pad26) -> DIS SDA
- DIS1 pad 27: unconnected-(DIS1-Pad27) -> DIS SCL
- DIS1 pad 30: unconnected-(DIS1-Pad30) -> VCC
- DIS1 pad 31: unconnected-(DIS1-Pad31) -> GND
- DIS1 pad 4: unconnected-(DIS1-Pad4) -> GND
- DIS1 pad 5: unconnected-(DIS1-Pad5) -> DSI1_D0_N
- DIS1 pad 6: unconnected-(DIS1-Pad6) -> DSI1_D0_P
- DIS1 pad 7: unconnected-(DIS1-Pad7) -> GND
- DIS1 pad 8: unconnected-(DIS1-Pad8) -> DSI1_D1_N
- DIS1 pad 9: unconnected-(DIS1-Pad9) -> DSI1_D1_P
- MK1 pad 3: unconnected-(MK1-Pad3) -> GND
- Module1 pad 107: GND -> unconnected-(Module1-Pad107)
- Module1 pad 108: GND -> unconnected-(Module1-Pad108)
- Module1 pad 113: GND -> unconnected-(Module1-Pad113)
- Module1 pad 114: GND -> unconnected-(Module1-Pad114)
- Module1 pad 119: GND -> unconnected-(Module1-Pad119)
- Module1 pad 120: GND -> unconnected-(Module1-Pad120)
- Module1 pad 125: GND -> unconnected-(Module1-Pad125)
- Module1 pad 126: GND -> unconnected-(Module1-Pad126)
- Module1 pad 128: unconnected-(Module1-Pad128) -> CAM_D0_N
- Module1 pad 130: unconnected-(Module1-Pad130) -> CAM_D0_P
- Module1 pad 131: GND -> unconnected-(Module1-Pad131)
- Module1 pad 132: GND -> unconnected-(Module1-Pad132)
- Module1 pad 134: unconnected-(Module1-Pad134) -> CAM_D1_N
- Module1 pad 136: unconnected-(Module1-Pad136) -> CAM_D1_P
- Module1 pad 137: GND -> unconnected-(Module1-Pad137)
- Module1 pad 138: GND -> unconnected-(Module1-Pad138)
- Module1 pad 140: unconnected-(Module1-Pad140) -> CAM_CK_N
- Module1 pad 142: unconnected-(Module1-Pad142) -> CAM_CK_P
- Module1 pad 144: GND -> unconnected-(Module1-Pad144)
- Module1 pad 150: GND -> unconnected-(Module1-Pad150)
- Module1 pad 155: GND -> unconnected-(Module1-Pad155)
- Module1 pad 156: GND -> unconnected-(Module1-Pad156)
- Module1 pad 161: GND -> unconnected-(Module1-Pad161)
- Module1 pad 162: GND -> unconnected-(Module1-Pad162)
- Module1 pad 167: GND -> unconnected-(Module1-Pad167)
- Module1 pad 168: GND -> unconnected-(Module1-Pad168)
- Module1 pad 173: GND -> unconnected-(Module1-Pad173)
- Module1 pad 174: GND -> unconnected-(Module1-Pad174)
- Module1 pad 175: unconnected-(Module1-Pad175) -> DSI1_D0_N
- Module1 pad 177: unconnected-(Module1-Pad177) -> DSI1_D0_P
- Module1 pad 179: GND -> unconnected-(Module1-Pad179)
- Module1 pad 180: GND -> unconnected-(Module1-Pad180)
- Module1 pad 181: unconnected-(Module1-Pad181) -> DSI1_D1_N
- Module1 pad 183: unconnected-(Module1-Pad183) -> DSI1_D1_P
- Module1 pad 185: GND -> unconnected-(Module1-Pad185)
- Module1 pad 186: GND -> unconnected-(Module1-Pad186)
- Module1 pad 187: unconnected-(Module1-Pad187) -> DSI1_C_N
- Module1 pad 189: unconnected-(Module1-Pad189) -> DSI1_C_P
- Module1 pad 191: GND -> unconnected-(Module1-Pad191)
- Module1 pad 192: GND -> unconnected-(Module1-Pad192)
- Module1 pad 193: unconnected-(Module1-Pad193) -> DSI1_D2_N
- Module1 pad 194: unconnected-(Module1-Pad194) -> DSI1_D3_N
- Module1 pad 195: unconnected-(Module1-Pad195) -> DSI1_D2_P
- Module1 pad 196: unconnected-(Module1-Pad196) -> DSI1_D3_P
- Module1 pad 197: GND -> unconnected-(Module1-Pad197)
- Module1 pad 28: unconnected-(Module1-Pad28) -> CODEC SCL
- Module1 pad 31: unconnected-(Module1-Pad31) -> CODEC SDA
- Module1 pad 37: unconnected-(Module1-Pad37) -> DIS SCL
- Module1 pad 39: unconnected-(Module1-Pad39) -> DIS SDA
- S1 pad 1: Net-(S1-Pad1) -> VCC
- S1 pad 2: Net-(S1-Pad1) -> VCC
- S1 pad 3: Net-(S1-Pad1) -> VCC
- S1 pad 4: Net-(S1-Pad1) -> Net-(BAT1-Pad1)
- S1 pad 5: PWR-KILL -> Net-(S1-Pad5)
- S1 pad 6: GPSGSM-SWITCH -> CAM-SWITCH
- S1 pad 7: CAM-SWITCH -> GPSGSM-SWITCH
- U5 pad 1: unconnected-(U5-Pad1) -> Net-(S1-Pad5)
- U5 pad 2: unconnected-(U5-Pad2) -> Net-(BAT1-Pad2)
- U5 pad 4: unconnected-(U5-Pad4) -> GND
- U8 pad 1: unconnected-(U8-Pad1) -> GND
- U8 pad 16: unconnected-(U8-Pad16) -> GND
- U8 pad 17: unconnected-(U8-Pad17) -> VCC
- U8 pad 18: unconnected-(U8-Pad18) -> GND
- U8 pad 2: unconnected-(U8-Pad2) -> VCC
- U8 pad 20: unconnected-(U8-Pad20) -> GND
- U8 pad 21: unconnected-(U8-Pad21) -> VCC
- U8 pad 24: unconnected-(U8-Pad24) -> VCC
- U8 pad 25: unconnected-(U8-Pad25) -> GND
- U8 pad 29: unconnected-(U8-Pad29) -> GND
- U8 pad 3: unconnected-(U8-Pad3) -> VCC
Routing:
- net D-: track 0.00 -> 23.4 mm
- net D+: track 0.00 -> 22.6 mm
Other:
- outline, holes or cut-outs redrawn
- board text added: "Caution, this device is a prototype. Compliance to norms is yet to be tested. Use at your own risk."
