File: EDA/cm4-carrier/cm4-carrier.kicad_sch (KiCad schematic)
At the start: 11 parts, among them J1 35RAPC4BHN2, J4 Conn_01x22_Female, J5 Conn_01x22_Female, J6 USB4105-GF-A, U1 Flash-LED-Lumiled

Commit message: update EDA files
Parts:
- added J2: FH72-31S-0.3SHW, SPIRIT-footprints:HRS_FH72-31S-0.3SHW, symbol SPIRIT-components:FH72-31S-0.3SHW
- added J3: 10pinFPC, SPIRIT-footprints:10PIN, symbol SPIRIT-components:10pinFPC
- added MK1: microphone, SPIRIT-footprints:microphone_SPH0645LM4H-B, symbol SPIRIT-components:microphone
- added SW1: VOL-, SPIRIT-footprints:buttonSW_TL3330_EWI, symbol SPIRIT-components:TL3330AF260QG
- added SW2: PROG, SPIRIT-footprints:buttonSW_TL3330_EWI, symbol SPIRIT-components:TL3330AF260QG
- added SW3: VOL+, SPIRIT-footprints:buttonSW_TL3330_EWI, symbol SPIRIT-components:TL3330AF260QG
- added SW4: POW, SPIRIT-footprints:buttonSW_TL3330_EWI, symbol SPIRIT-components:TL3330AF260QG
Other:
- note added: "DIS22"
- note added: "DIS31"
- note removed: "DIS"

Commit message: update files
Parts:
- removed J4: Conn_01x22_Female, SPIRIT-footprints:Hirose_FH12-22S-0.5SH_1x22-1MP_P0.50mm_Horizontal, symbol Connector:Conn_01x22_Female
- added B1: VIBR, SPIRIT-footprints:VIBRATION-PUI_HD-EMB1205-3-SC-R, symbol SPIRIT-components:VIBR
- added U2: CHARGER-BQ24161YFFR, SPIRIT-footprints:CHARGER-YFF49, symbol SPIRIT-components:CHARGER-BQ24161YFFR
- added U3: BAT-MONITOR-BQ27530YZFT-G1, SPIRIT-footprints:BAT-MONITOR-YZF15_TEX, symbol SPIRIT-components:BAT-MONITOR-BQ27530YZFT-G1
- added U4: STABILIZER-MC34063ADR, SPIRIT-footprints:STABILIZER-MC34063ADR, symbol SPIRIT-components:STABILIZER-MC34063ADR
- added U5: BAT-CONNECTOR-FLTS22WR00, SPIRIT-footprints:BAT-CONNECTOR-FLTS22WR00, symbol SPIRIT-components:BAT-CONNECTOR-FLTS22WR00
- added U6: GPS-moduleYIC31009EBGG, SPIRIT-footprints:GPS-moduleYIC31009EBGG, symbol SPIRIT-components:GPS-moduleYIC31009EBGG
- J5: renamed from J3; value 10pinFPC -> FINGER
- renumbered J5 to J1, J6 to J2, J2 to J3, J1 to J4, LS3 to LS1, LS4 to LS2
Other:
- note added: "DIS"
- note removed: "DIS22"
- note removed: "DIS31"
- moved on the sheet: J1, J3, J5, R1

Commit message: update EDA
Parts:
- removed J4: 35RAPC4BHN2, SPIRIT-footprints:35mm-jack-35RAPC4BHN2-switchcraft, symbol SPIRIT-components:35RAPC4BHN2
- removed U2: CHARGER-BQ24161YFFR, SPIRIT-footprints:CHARGER-YFF49, symbol SPIRIT-components:CHARGER-BQ24161YFFR
- removed U4: STABILIZER-MC34063ADR, SPIRIT-footprints:STABILIZER-MC34063ADR, symbol SPIRIT-components:STABILIZER-MC34063ADR
- removed U6: GPS-moduleYIC31009EBGG, SPIRIT-footprints:GPS-moduleYIC31009EBGG, symbol SPIRIT-components:GPS-moduleYIC31009EBGG
- added D1: LED-INDICATOR, SPIRIT-footprints:LED-INDICATOR, symbol SPIRIT-components:LED-INDICATOR
- added J4: 35mmJACK-TRRS, SPIRIT-footprints:35mmJACK-TRRS, symbol SPIRIT-components:35mmJACK-TRRS
- added J6: SIM-G85D1160022HHR, SPIRIT-footprints:SIM-AMPHENOL_G85D1160022HHR, symbol SPIRIT-components:SIM-G85D1160022HHR
- added S1: DIPSWITCH, SPIRIT-footprints:DIPSWITC-SW_219-4MST, symbol SPIRIT-components:DIPSWITCH219-4MST
- added U2: CHARGER-SWITCHER-BQ25303JRTER, SPIRIT-footprints:CHARGER-SWITCHER-RTE0016C, symbol SPIRIT-components:CHARGER-SWITCHER-BQ25303JRTER
- added U4: BAT-STEP-UP-MIC2876-5.0YMT-TR, SPIRIT-footprints:BAT-STEP-UP-UDFN8_2X2_MCH, symbol SPIRIT-components:BAT-STEP-UP-MIC2876-5.0YMT-TR
- added U6: GSM-GPS-EC25VFA-512-STD, SPIRIT-footprints:GSM-GPS-XCVR_EC25VFA-512-STD, symbol SPIRIT-components:GSM-GPS-EC25VFA-512-STD
- added U8: DAC-TLV320DAC3100IRHBR, SPIRIT-footprints:DAC-IC_ADS125H01IRHBT, symbol SPIRIT-components:DAC-TLV320DAC3100IRHBR
Connections:
- net at U5.1 (BAT+): now also S1.5
- net at MK1.5 (VDD): now also S1.8
Other:
- moved on the sheet: MK1, U3, U5

Commit message: update EDA
Parts:
- removed BAT1: battery-37V2AhLP504783JU, SPIRIT-footprints:battery-37V2AhLP504783JU, symbol SPIRIT-components:battery-37V2AhLP504783JU
- removed J1: Conn_01x22_Female, SPIRIT-footprints:Hirose_FH12-22S-0.5SH_1x22-1MP_P0.50mm_Horizontal, symbol Connector:Conn_01x22_Female
- removed J4: 35mmJACK-TRRS, SPIRIT-footprints:35mmJACK-TRRS, symbol SPIRIT-components:35mmJACK-TRRS
- added BAT?: battery-37V2AhLP504783JU, SPIRIT-footprints:battery-37V2AhLP504783JU, symbol SPIRIT-components:battery-37V2AhLP504783JU
- added J1: SJ2-35894B-SMT-TR, SPIRIT-footprints:35mmJACK-CUI_SJ2-35894B-SMT-TR, symbol SPIRIT-components:SJ2-35894B-SMT-TR
- added J3: CAM FPC15pins05pitch, SPIRIT-footprints:FPC15pins05pitch, symbol SPIRIT-components:FPC15pins05pitch
- added R2, R3: 5.1kOhm, SPIRIT-footprints:CC-PULLDOWN-RESISOTR, symbol SPIRIT-components:CC-PULLDOWN-RESISTOR
- renumbered J3 to DIS1
Connections:
- net D+: now also J2.B6 (DP2)
- net D-: now also J2.B7 (DN2)
- net GND: now also B1.N, J2.B1_A12 (GND__1), J2.SH1 (SHELL_GND), J2.SH2 (SHELL_GND__1), J2.SH3 (SHELL_GND__2), J2.SH4 (SHELL_GND__3), J6.C5 (GND), J6.S1 (SHIELD_GND), J6.S2 (SHIELD_GND__1), J6.S3 (SHIELD_GND__2), MK1.3 (GND), Module1.1 (GND), Module1.13 (GND), Module1.14 (GND), Module1.198 (GND), Module1.2 (GND), Module1.22 (GND), Module1.23 (GND), Module1.32 (GND), Module1.33 (GND), Module1.42 (GND), Module1.43 (GND), Module1.52 (GND), Module1.53 (GND), Module1.60 (GND), Module1.66 (GND), Module1.71 (GND), Module1.74 (GND), Module1.8 (GND), Module1.98 (GND), U1.1 (-), J3.1, J3.10, J3.4, R2.1, R3.2; no longer Module1.107 (GND)
- net VCC: now reaches SW2.1
- net VCC: now also S1.1, S1.2, S1.3, SW1.1, SW3.1, SW4.1
- net at SW2.2: now also Module1.50 (GPIO17)
- net at SW1.2: now also Module1.54 (GPIO4)
- net CAM_D0_N: now reaches Module1.128 (CAM0_D0_N)
- net CAM_D0_N: now also J3.2
- net CAM_D0_P: now reaches Module1.130 (CAM0_D0_P)
- net CAM_D0_P: now also J3.3
- net CAM_D1_N: now reaches Module1.134 (CAM0_D1_N)
- net CAM_D1_N: now also J3.5
- net CAM_D1_P: now reaches Module1.136 (CAM0_D1_P)
- net CAM_D1_P: now also J3.6
- net CAM_CK_N: now reaches Module1.140 (CAM0_C_N)
- net CAM_CK_N: now also J3.8
- net CAM_CK_P: now reaches Module1.142 (CAM0_C_P)
- net CAM_CK_P: now also J3.9
- net at U1.2 (+): now also Module1.46 (GPIO22)
- net at Module1.48 (GPIO27): now also B1.P
- net at Module1.56 (GPIO3): now also SW3.2
- net at Module1.58 (GPIO2): now also SW4.2
- net at CR1.1: now also J2.A4_B9 (VBUS), J2.B4_A9 (VBUS__1)
- net CAM-SWITCH: now reaches S1.6
- net CAM-SWITCH: now also J3.15
- net GPSGSM-SWITCH: now reaches S1.7
- net MIC-SWITCH: now reaches MK1.5 (VDD), S1.8
- net at J2.A5 (CC1): now also R2.2
- net at J2.B5 (CC2): now also R3.1
- new net CAM_SCL: J3.13
- new net CAM_SDA: J3.14
- new net JACK-IN: J1.10
- no-connect marks 0 -> 6
Other:
- note added: "3.3V"
- note added: "Audio"
- note added: "GSM & GPS"
- note added: "Other"
- note added: "Power"
- note removed: "CAM"
- note removed: "DIS"
- moved on the sheet: B1, CR1, D1, DIS1, J2, J5, J6, LS1, LS2, MK1, Module1A, Module1B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

Commit message: update EDA
Parts:
- removed CR1: SMBJ5.0A, SPIRIT-footprints:TVS-DO-214AASMB_J-BEND_LTF, symbol SPIRIT-components:SMBJ5.0A
- removed J3: CAM FPC15pins05pitch, SPIRIT-footprints:FPC15pins05pitch, symbol SPIRIT-components:FPC15pins05pitch
- added TP1, TP2, TP3, TP4, TP5, TP6: test-pad-1, SPIRIT-footprints:test-pad-1, symbol SPIRIT-components:test-pad-1
- added U10: TVSdiode-array-TPD4EUSB30DQAR, SPIRIT-footprints:TVSdiode-arrayDQA10, symbol SPIRIT-components:TVSdiode-array-TPD4EUSB30DQAR
- added U7: FPC15pin-1mm-pitch-F52Q-1A7H1-11015, SPIRIT-footprints:FPC15pin-1mm-pitch-CONN_F52Q-1A7H1-11015_AMP, symbol SPIRIT-components:FPC15pin-1mm-pitch-F52Q-1A7H1-11015
- added U9: CODEC-TLV320AIC3204IRHBR, SPIRIT-footprints:CODEC-QFN50P500X500X100-33N, symbol SPIRIT-components:CODEC-TLV320AIC3204IRHBR
- gave numbers to parts that had none: 1
Connections:
- net CAM-SWITCH: now also TP1.1 (A), U7.15
- net CAM_CK_N: now also U7.8
- net CAM_CK_P: now also U7.9
- net CAM_D0_N: now also U7.2
- net CAM_D0_P: now also U7.3
- net CAM_D1_N: now also U7.5
- net CAM_D1_P: now also U7.6
- net CAM_IO0: now also TP2.1 (A), U7.11
- net CAM_SCL: now also U7.13
- net CAM_SDA: now also U7.14
- net D+: now also U10.1 (D1+)
- net D-: now also U10.2 (D1-)
- net GND: now also DIS1.1, DIS1.10, DIS1.13, DIS1.16, DIS1.19, DIS1.20, DIS1.31, DIS1.4, DIS1.7, U5.4 (OUT-), U8.1 (IOVSS), U8.16 (AVSS), U8.18 (DVSS), U8.20 (SPKVSS), U8.25 (SPKVSS__1), U8.29 (HPVSS), U10.3 (GND), U10.8 (GND), U7.1, U7.10, U7.4, U9.17 (AVSS), U9.28 (DVSS), U9.7 (IOVSS)
- net VCC: now also DIS1.25, DIS1.30, U8.17 (AVDD), U8.2 (IOVDD), U8.21 (SPKVDD), U8.24 (SPKVDD__1), U8.3 (DVDD), U9.24 (AVDD)
- net DSI1_D0_N: now reaches Module1.175 (DSI1_D0_N)
- net DSI1_D0_N: now also DIS1.5
- net DSI1_D0_P: now reaches Module1.177 (DSI1_D0_P)
- net DSI1_D0_P: now also DIS1.6
- net DSI1_D1_N: now reaches Module1.181 (DSI1_D1_N)
- net DSI1_D1_N: now also DIS1.8
- net DSI1_D1_P: now reaches Module1.183 (DSI1_D1_P)
- net DSI1_D1_P: now also DIS1.9
- net DSI1_C_N: now reaches Module1.187 (DSI1_C_N)
- net DSI1_C_N: now also DIS1.11
- net DSI1_C_P: now reaches Module1.189 (DSI1_C_P)
- net DSI1_C_P: now also DIS1.12
- net DSI1_D2_N: now reaches Module1.193 (DSI1_D2_N)
- net DSI1_D2_N: now also DIS1.14
- net DSI1_D3_N: now reaches Module1.194 (DSI1_D3_N)
- net DSI1_D3_N: now also DIS1.17
- net DSI1_D2_P: now reaches Module1.195 (DSI1_D2_P)
- net DSI1_D2_P: now also DIS1.15
- net DSI1_D3_P: now reaches Module1.196 (DSI1_D3_P)
- net DSI1_D3_P: now also DIS1.18
- net at Module1.46 (GPIO22), U1.2 (+): now also TP3.1 (A)
- net CODEC SCL: now reaches Module1.28 (GPIO13)
- net CODEC SCL: now also U9.9 (SCL/~{SS})
- net CODEC SDA: now reaches Module1.31 (GPIO12)
- net CODEC SDA: now also U9.10 (SDA/MOSI)
- net DIS SCL: now reaches Module1.37 (GPIO7)
- net DIS SCL: now also DIS1.27
- net DIS SDA: now reaches Module1.39 (GPIO8)
- net DIS SDA: now also DIS1.26
- net at B1.P, Module1.48 (GPIO27): now also TP4.1 (A)
- net USBC POW: now reaches J2.A4_B9 (VBUS), J2.B4_A9 (VBUS__1)
- net USBC POW: now also U10.5 (D2-)
- net at S1.4: now also BAT1.1 (+)
- net at BAT1.2 (-): now also U5.2 (BAT-)
- no-connect marks 6 -> 18
Other:
- note added: "(remove if not enough gpio)"
- note added: "2.8V lin. reg. needed"
- note added: "35mm Jack should be ESD protected come back to this task when USB 3.0 implemented"
- note added: "Camera"
- note added: "I think I also need an ADC for the headphone mic"
- note added: "LEFT"
- note added: "RIGHT"
- note added: "Sreen"
- note added: "USB C"
- note added: "any leftover gpio"
- note added: "consider changing the bat monitor to regular SMD to avoid mixing with BGA"
- note added: "make sure the connector is in the correct posistion relative to the screen (like in case of the camera)"
- note added: "maybe do 2 separate step ups for 3.3V 5V"
- note added: "maybe the bat monitor isn't needed?"
- note added: "should there be a separate GND and power source for heaphones (for audiophiles)?"
- note added: "these pins need to be connected to any remaining GPIO"
- note added: "this switch should probably be changed to 90deg switches for accesibility reasons"
- note added: "~22V step up needed"
- moved on the sheet: B1, BAT1, D1, J1, J2, J5, J6, LS1, LS2, MK1, Module1A, Module1B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
