File: EDA/cm4-carrier-kicad8/cm4-carrier.kicad_pcb (KiCad board)
At the start: 2 copper layers, 80 x 148.2 mm, 41 parts, among them J1 SJ2-35894B-SMT-TR, J2 USB4105-GF-A, J5 FINGER, J6 SIM-G85D1160022HHR, SW1 VOL-, SW2 PROG, SW3 VOL+, SW4 POW, U1 Flash-LED-Lumiled, U10 TVSdiode-array-TPD4EUSB30DQAR, U2 CHARGER-SWITCHER-BQ25303JRTER, U3 BAT-MONITOR-BQ27530YZFT-G1, U4 BAT-STEP-UP-MIC2876-5.0YMT-TR, U5 BAT-CONNECTOR-FLTS22WR00, U6 GSM-GPS-EC25VFA-512-STD, U7 FPC15pin-1mm-pitch-F52Q-1A7H1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, U8 DAC-TLV320DAC3100IRHBR, U9 CODEC-TLV320AIC3204IRHBR

Commit message: update EDA
Parts:
- added J3: USB4056-03-A, SPIRIT-footprints:USBC3-2, F.Cu at (93.8, 169.8)
- added SBU1: test-pad-1, SPIRIT-footprints:test-pad-1, F.Cu at (104.0, 173.0)
- added SBU2: test-pad-1, SPIRIT-footprints:test-pad-1, F.Cu at (104.0, 175.5)
- added logo1: KiCad-Logo2_5mm_SilkScreen, Symbol:KiCad-Logo2_5mm_SilkScreen, F.Cu at (65.0, 101.5)
- moved S1 103.2 mm to (-38.2, 125.2)
- moved R1 69.6 mm to (-30.2, 113.5)
- moved J2 20.2 mm to (110.5, 189.5)
- moved R2 0.47 mm to (90.0, 175.9)
- moved R3 0.47 mm to (90.0, 172.2)
- moved J1 0.46 mm to (67.0, 170.4)
Connections:
- J2 pad A4_B9: Net-(J2-PadA4_B9) -> USBC POW
- J2 pad B4_A9: Net-(J2-PadA4_B9) -> USBC POW
- U10 pad 4: D+ -> unconnected-(U10-D2+-Pad4)
- U10 pad 5: D- -> USBC POW
Routing:
- net D-: track 23.4 -> 0.00 mm
- net D+: track 22.6 -> 0.00 mm

Commit message: finish USB C kicad 8
Parts:
- removed J2: USB4105-GF-A, SPIRIT-footprints:USB_C_GCT_USB4105-GF-A
- removed U10: TVSdiode-array-TPD4EUSB30DQAR, SPIRIT-footprints:TVSdiode-arrayDQA10
- added C1: 0.33 µF coupling cap, SPIRIT-footprints:USBC_capacitor_CAPC0603X33N, F.Cu at (100.2, 155.2)
- added C2: 0.33 µF coupling cap, SPIRIT-footprints:USBC_capacitor_CAPC0603X33N, F.Cu at (100.2, 157.1)
- added C3: 0.33 µF coupling cap, SPIRIT-footprints:USBC_capacitor_CAPC0603X33N, F.Cu at (100.2, 159.1)
- added C4: 0.33 µF coupling cap, SPIRIT-footprints:USBC_capacitor_CAPC0603X33N, F.Cu at (100.2, 161.0)
- added TVS-PUSB3FR1: ~, SPIRIT-footprints:TVS-array-IC_PUSB3AB6Z, F.Cu at (104.6, 167.0)
- added ZD1: protection-PESD5V0C1USFYL, SPIRIT-footprints:USB-ESD-protection-diode-PESD5V0C1USFYL-SOD962-2_DSN0603-2_NEX, F.Cu at (103.7, 158.0)
- moved S1 105.7 mm to (65.2, 147.2)
- moved R1 74.5 mm to (41.7, 133.0)
- renumbered SBU1 to TP7, SBU2 to TP8
Connections:
- J3 pad A10: unconnected-(J3-PadA10) -> RX1-
- J3 pad A11: unconnected-(J3-PadA11) -> RX1+
- J3 pad A2: unconnected-(J3-PadA2) -> TX1+
- J3 pad A3: unconnected-(J3-PadA3) -> TX1-
- J3 pad B10: unconnected-(J3-PadB10) -> RX1-
- J3 pad B11: unconnected-(J3-PadB11) -> RX1+
- J3 pad B2: unconnected-(J3-PadB2) -> TX1+
- J3 pad B3: unconnected-(J3-PadB3) -> TX1-
- U6 pad 100: unconnected-(U6-GND__29-Pad100) -> GND
- U6 pad 101: unconnected-(U6-GND__30-Pad101) -> GND
- U6 pad 102: unconnected-(U6-GND__31-Pad102) -> GND
- U6 pad 103: unconnected-(U6-GND__32-Pad103) -> GND
- U6 pad 104: unconnected-(U6-GND__33-Pad104) -> GND
- U6 pad 105: unconnected-(U6-GND__34-Pad105) -> GND
- U6 pad 106: unconnected-(U6-GND__35-Pad106) -> GND
- U6 pad 107: unconnected-(U6-GND__36-Pad107) -> GND
- U6 pad 108: unconnected-(U6-GND__37-Pad108) -> GND
- U6 pad 109: unconnected-(U6-GND__38-Pad109) -> GND
- U6 pad 110: unconnected-(U6-GND__39-Pad110) -> GND
- U6 pad 111: unconnected-(U6-GND__40-Pad111) -> GND
- U6 pad 112: unconnected-(U6-GND__41-Pad112) -> GND
- U6 pad 19: unconnected-(U6-GND__2-Pad19) -> GND
- U6 pad 22: unconnected-(U6-GND__3-Pad22) -> GND
- U6 pad 36: unconnected-(U6-GND__4-Pad36) -> GND
- U6 pad 46: unconnected-(U6-GND__5-Pad46) -> GND
- U6 pad 48: unconnected-(U6-GND__6-Pad48) -> GND
- U6 pad 50: unconnected-(U6-GND__7-Pad50) -> GND
- U6 pad 51: unconnected-(U6-GND__8-Pad51) -> GND
- U6 pad 52: unconnected-(U6-GND__9-Pad52) -> GND
- U6 pad 53: unconnected-(U6-GND__10-Pad53) -> GND
- U6 pad 54: unconnected-(U6-GND__11-Pad54) -> GND
- U6 pad 56: unconnected-(U6-GND__12-Pad56) -> GND
- U6 pad 72: unconnected-(U6-GND__13-Pad72) -> GND
- U6 pad 8: unconnected-(U6-GND-Pad8) -> GND
- U6 pad 85: unconnected-(U6-GND__14-Pad85) -> GND
- U6 pad 86: unconnected-(U6-GND__15-Pad86) -> GND
- U6 pad 87: unconnected-(U6-GND__16-Pad87) -> GND
- U6 pad 88: unconnected-(U6-GND__17-Pad88) -> GND
- U6 pad 89: unconnected-(U6-GND__18-Pad89) -> GND
- U6 pad 9: unconnected-(U6-GND__1-Pad9) -> GND
- U6 pad 90: unconnected-(U6-GND__19-Pad90) -> GND
- U6 pad 91: unconnected-(U6-GND__20-Pad91) -> GND
- U6 pad 92: unconnected-(U6-GND__21-Pad92) -> GND
- U6 pad 93: unconnected-(U6-GND__22-Pad93) -> GND
- U6 pad 94: unconnected-(U6-GND__23-Pad94) -> GND
- U6 pad 95: unconnected-(U6-GND__24-Pad95) -> GND
- U6 pad 96: unconnected-(U6-GND__25-Pad96) -> GND
- U6 pad 97: unconnected-(U6-GND__26-Pad97) -> GND
- U6 pad 98: unconnected-(U6-GND__27-Pad98) -> GND
- U6 pad 99: unconnected-(U6-GND__28-Pad99) -> GND
