File: EDA/cm4-carrier-kicad8/cm4-carrier.kicad_sch (KiCad schematic)
At the start: 36 parts, among them J1 SJ2-35894B-SMT-TR, J2 USB4105-GF-A, J5 FINGER, J6 SIM-G85D1160022HHR, SW1 VOL-, SW2 PROG, SW3 VOL+, SW4 POW, U1 Flash-LED-Lumiled, U10 TVSdiode-array-TPD4EUSB30DQAR, U2 CHARGER-SWITCHER-BQ25303JRTER, U3 BAT-MONITOR-BQ27530YZFT-G1, U4 BAT-STEP-UP-MIC2876-5.0YMT-TR, U5 BAT-CONNECTOR-FLTS22WR00, U6 GSM-GPS-EC25VFA-512-STD, U7 FPC15pin-1mm-pitch-F52Q-1A7H1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, U8 DAC-TLV320DAC3100IRHBR, U9 CODEC-TLV320AIC3204IRHBR

Commit message: update EDA
Parts:
- removed J2: USB4105-GF-A, SPIRIT-footprints:USB_C_GCT_USB4105-GF-A, symbol USB_C_SPIRIT:USB4105-GF-A
- removed R2, R3: 5.1kOhm, SPIRIT-footprints:CC-PULLDOWN-RESISOTR, symbol SPIRIT-components:CC-PULLDOWN-RESISTOR
- added J3: USB4056-03-A, SPIRIT-footprints:USBC3-2, symbol SPIRIT-components:USB4056-03-A
- added TP7, TP8: test-pad-1, SPIRIT-footprints:test-pad-1, symbol SPIRIT-components:test-pad-1
Connections:
- net D+: now also J3.A6, J3.B6
- net D-: now also J3.A7, J3.B7
- net GND: now also J3.A1, J3.A12, J3.B1, J3.B12
- net USBC POW: now also J3.A4, J3.A9, J3.B4, J3.B9; no longer U10.5 (D2-)
- new net: J3.A8, TP7.1 (A)
- new net: J3.B8, TP8.1 (A)
- new net CC1: J3.A5
- new net CC2: J3.B5
- no-connect marks 18 -> 17
Other:
- note added: "(Not important. Remove if not enough gpio to use it.)"
- note added: "ADD TVS diodes IC and singular diodes"
- note added: "Probably the DAC can be deleted. I think the codec works as a DAC and ADC"
- note added: "USB C 3.0"
- note added: "consider changing the bat monitor to regular SMD to avoid BGA components. Perhaps it is better to have only SMD and not mix mounting types. This will probably make assembly easier"
- note removed: "(remove if not enough gpio)"
- note removed: "I think I also need an ADC for the headphone mic"
- note removed: "USB C"
- note removed: "consider changing the bat monitor to regular SMD to avoid mixing with BGA"
- note removed: "this switch should probably be changed to 90deg switches for accesibility reasons"
- moved on the sheet: U10

Commit message: finish USB C kicad 8
Parts:
- removed U10: TVSdiode-array-TPD4EUSB30DQAR, SPIRIT-footprints:TVSdiode-arrayDQA10, symbol SPIRIT-components:TVSdiode-array-TPD4EUSB30DQAR
- added C1, C2, C3, C4: 0.33 µF coupling cap, SPIRIT-footprints:USBC_capacitor_CAPC0603X33N, symbol SPIRIT-components:USBC_capacitor_GRM033R60J334ME90D
- added TVS-PUSB3FR1: ~, SPIRIT-footprints:TVS-array-IC_PUSB3AB6Z, symbol SPIRIT-components:TVS-diode-array-PUSB3FR6
- added ZD1: protection-PESD5V0C1USFYL, SPIRIT-footprints:USB-ESD-protection-diode-PESD5V0C1USFYL-SOD962-2_DSN0603-2_NEX, symbol SPIRIT-components:USB-protection-diode-PESD5V0C1USFYL
Connections:
- net D+: now also TVS-PUSB3FR1.5 (D+)
- net D-: now also TVS-PUSB3FR1.4 (D-)
- net GND: now also U6.100 (GND__29), U6.101 (GND__30), U6.102 (GND__31), U6.103 (GND__32), U6.104 (GND__33), U6.105 (GND__34), U6.106 (GND__35), U6.107 (GND__36), U6.108 (GND__37), U6.109 (GND__38), U6.110 (GND__39), U6.111 (GND__40), U6.112 (GND__41), U6.19 (GND__2), U6.22 (GND__3), U6.36 (GND__4), U6.46 (GND__5), U6.48 (GND__6), U6.50 (GND__7), U6.51 (GND__8), U6.52 (GND__9), U6.53 (GND__10), U6.54 (GND__11), U6.56 (GND__12), U6.72 (GND__13), U6.8 (GND), U6.85 (GND__14), U6.86 (GND__15), U6.87 (GND__16), U6.88 (GND__17), U6.89 (GND__18), U6.9 (GND__1), U6.90 (GND__19), U6.91 (GND__20), U6.92 (GND__21), U6.93 (GND__22), U6.94 (GND__23), U6.95 (GND__24), U6.96 (GND__25), U6.97 (GND__26), U6.98 (GND__27), U6.99 (GND__28), TVS-PUSB3FR1.2 (GND), ZD1.2
- net USBC POW: now also ZD1.1
- net RX1-: now reaches J3.A10
- net RX1-: now also J3.B10, TVS-PUSB3FR1.6 (Rx-)
- net RX1+: now reaches J3.A11
- net RX1+: now also J3.B11, TVS-PUSB3FR1.7 (RX+)
- net TX1+: now reaches J3.A2
- net TX1+: now also J3.B2, TVS-PUSB3FR1.3 (Tx+)
- net TX1-: now reaches J3.A3
- net TX1-: now also J3.B3, TVS-PUSB3FR1.1 (Tx-)
- no-connect marks 17 -> 16
Other:
- note added: "RX1"
- note added: "RX2"
- note added: "TX1"
- note added: "TX2"
- note added: "is it ok to connet all of these pins to the same GND?"
- note added: "make sure the connector is in the correct posistion relative to the screen (like in case of the camera). Also make sure the cable doesn't have to bend to much"
- note added: "todo add capacitors on tx and rx"
- note added: "todo connect tx and rx pins to CM5"
- note removed: "ADD TVS diodes IC and singular diodes"
- note removed: "make sure the connector is in the correct posistion relative to the screen (like in case of the camera)"
- moved on the sheet: J3, R1, TP7, TP8
